Commit message: Remove fingertip collisions from urdf

File: trajectory_planning/robot/panda_description/panda_ec.urdf (robot description, URDF)
Before this commit: robot panda_ec, 12 links, 11 joints
Links:
- link panda_leftfinger: geometry visual mesh filename=finger.dae
- link panda_rightfinger: geometry visual mesh filename=finger.dae

File: trajectory_planning/robot/panda_description/panda_sc.urdf (robot description, URDF)
Before this commit: robot panda, 12 links, 11 joints
Links:
- link panda_leftfinger: geometry visual mesh filename=finger.dae
- link panda_rightfinger: geometry visual mesh filename=finger.dae
